File: Board/video_board.brd (EAGLE design)
At the start: 110 x 70 mm, 83 parts, among them IC1 74HCT04, IC2 CXA1645, Q1 4,43Mhz, Q2 3,58Mhz, T1 2SC1815, T2 2SC1815, T3 2SC1815, T4 2SC1815, X2 DIN-8

Commit message: Latest fixes for schematics and partslist
Fixed incorrect C8 value in partslist and schematics
Parts:
- C8: value 10 mF -> 10 uF
Changed lines of the file:
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@@
 <element name="C5" library="rcl" package="SMC_B" value="10 uF" x="92" y="17" smashed="yes" rot="R180"/>
 <element name="R6" library="resistor" package="R0805" value="750 Ohm" x="30" y="21" smashed="yes" rot="R90"/>
-<element name="C8" library="rcl" package="SMC_B" value="10 mF" x="30" y="15" smashed="yes" rot="R270"/>
+<element name="C8" library="rcl" package="SMC_B" value="10 uF" x="30" y="15" smashed="yes" rot="R270"/>
 <element name="R2" library="resistor" package="R0805" value="22 kOhm" x="51" y="20" smashed="yes" rot="R180"/>
 <element name="R4" library="resistor" package="R0805" value="10 kOhm" x="75" y="29" smashed="yes" rot="R270"/>
